File: board/ir-train-detector.kicad_pcb (KiCad board)
At the start: 2 copper layers, 107 parts, among them J1 ST_01x02, J10 IR_MOD1, J11 IR_MOD1, J2 JTAG, J3 BSL_SEL, J4 USB_B, J6 IR_MOD1, J7 IR_MOD1, J8 IR_MOD1, J9 IR_MOD1, Q1 AO3407A, Q2 AO3407A, Q3 AO3407A, Q4 AO3407A, Q5 AO3407A, Q6 AO3407A, SW1 SW_Push, U1 AP63300WU, U2 FT231XS, U3 MSP430G2553IPW28, U4 LM358, U5 LM324A, Y1 32768Hz

Commit message: board layout
Parts:
- removed the R7 at (115.0, 74.2)
- removed the R7 at (92.5, 47.3)
- removed the R8 at (67.2, 101.5)
- removed the R8 at (86.4, 50.7)
- added D11: LED, LED_SMD:LED_0603_1608Metric_Pad1.05x0.95mm_HandSolder, F.Cu at (101.0, 81.0)
- added H1: MountingHole, MountingHole:MountingHole_3.2mm_M3_DIN965, F.Cu at (95.0, 62.5)
- added H2: MountingHole, MountingHole:MountingHole_3.2mm_M3_DIN965, F.Cu at (217.8, 79.5)
- added H3: MountingHole, MountingHole:MountingHole_3.2mm_M3_DIN965, F.Cu at (168.5, 55.2)
- added J5: Screw_Terminal_01x07, TerminalBlock_RND:TerminalBlock_RND_205-00006_1x07_P5.00mm_Horizontal, F.Cu at (159.4, 81.2)
- added R49: 10k, Resistor_SMD_AKL:R_0603_1608Metric_Pad1.05x0.95mm_HandSolder, F.Cu at (220.5, 60.5)
- added R7: 470R, Resistor_SMD_AKL:R_0603_1608Metric_Pad1.05x0.95mm_HandSolder, F.Cu at (154.5, 75.8)
- added R8: 470k, Resistor_SMD_AKL:R_0603_1608Metric_Pad1.05x0.95mm_HandSolder, F.Cu at (187.8, 65.5)
- added TP1: TestPoint, TestPoint:TestPoint_Pad_D1.5mm, F.Cu at (133.0, 65.2)
- added TP10: TestPoint, TestPoint:TestPoint_Pad_D1.5mm, F.Cu at (155.2, 62.4)
- added TP2: TestPoint, TestPoint:TestPoint_Pad_D1.5mm, F.Cu at (182.4, 60.6)
- added TP3: TestPoint, TestPoint:TestPoint_Pad_D1.5mm, F.Cu at (113.2, 62.2)
- added TP4: TestPoint, TestPoint:TestPoint_Pad_D1.5mm, F.Cu at (177.6, 61.8)
- added TP5: TestPoint, TestPoint:TestPoint_Pad_D1.5mm, F.Cu at (176.6, 64.8)
- added TP6: TestPoint, TestPoint:TestPoint_Pad_D1.5mm, F.Cu at (112.5, 82.5)
- added TP7: TestPoint, TestPoint:TestPoint_Pad_D1.5mm, F.Cu at (119.0, 83.5)
- added TP8: TestPoint, TestPoint:TestPoint_Pad_D1.5mm, F.Cu at (115.8, 76.8)
- added TP9: TestPoint, TestPoint:TestPoint_Pad_D1.5mm, F.Cu at (114.5, 79.5)
- C1: value 470u -> 100n; footprint Capacitor_THT_AKL:CP_Radial_D12.5mm_P5.00mm -> Capacitor_SMD_Handsoldering_AKL:C_0603_1608Metric
- C11, C7: value 100n -> 33n
- C12: value 4u7 -> 100n
- C13: value 47p -> 100n; footprint Capacitor_SMD_Handsoldering_AKL:C_0805_2012Metric -> Capacitor_SMD_Handsoldering_AKL:C_0603_1608Metric
- C14: value 47p -> 10u; footprint Capacitor_SMD_Handsoldering_AKL:C_0805_2012Metric -> Capacitor_SMD_Handsoldering_AKL:C_1206_3216Metric
- C15: value 2n2 -> 100n
- C18: value 33n -> 4u7; footprint Capacitor_SMD_Handsoldering_AKL:C_0603_1608Metric -> Capacitor_THT_AKL:CP_Radial_D4.0mm_P1.50mm
- C2: value 10u -> 56p; footprint Capacitor_SMD_Handsoldering_AKL:C_1206_3216Metric -> Capacitor_SMD_Handsoldering_AKL:C_0805_2012Metric
- C20: value 33n -> 2n2; footprint Capacitor_SMD_Handsoldering_AKL:C_0603_1608Metric -> Capacitor_SMD_Handsoldering_AKL:C_0805_2012Metric
- C3: value 100n -> 22u; footprint Capacitor_SMD_Handsoldering_AKL:C_0603_1608Metric -> Capacitor_SMD_Handsoldering_AKL:C_1206_3216Metric
- C4: value 56p -> 22u; footprint Capacitor_SMD_Handsoldering_AKL:C_0603_1608Metric -> Capacitor_SMD_Handsoldering_AKL:C_1206_3216Metric
- C5: value 22u -> 470u; footprint Capacitor_SMD_Handsoldering_AKL:C_0805_2012Metric -> Capacitor_THT_AKL:CP_Radial_D10.0mm_P5.00mm
- C6: value 22u -> 10u; footprint Capacitor_SMD_Handsoldering_AKL:C_0805_2012Metric -> Capacitor_SMD_Handsoldering_AKL:C_1206_3216Metric
- C8: value 100n -> 47p; footprint Capacitor_SMD_Handsoldering_AKL:C_0603_1608Metric -> Capacitor_SMD_Handsoldering_AKL:C_0805_2012Metric
- C9: value 10u -> 47p; footprint Capacitor_SMD_Handsoldering_AKL:C_1206_3216Metric -> Capacitor_SMD_Handsoldering_AKL:C_0805_2012Metric
- D1: value AB05S -> LED; footprint Diode_SMD_Handsoldering_AKL:Diode_Bridge_Diotec_ABS -> LED_SMD:LED_0603_1608Metric_Pad1.05x0.95mm_HandSolder
- D2: value LED -> AB05S; footprint LED_SMD:LED_0603_1608Metric_Pad1.05x0.95mm_HandSolder -> Diode_SMD_Handsoldering_AKL:Diode_Bridge_Diotec_ABS
- D3: value LED -> LED_PWR
- D9: value LED_PWR -> LED
- J1: footprint Resistor_SMD_AKL:R_0603_1608Metric_Pad1.05x0.95mm_HandSolder -> TerminalBlock_RND:TerminalBlock_RND_205-00001_1x02_P5.00mm_Horizontal
- J10, J11, J6, J9: value IR_MOD1 -> Screw_Terminal_01x03; footprint Connector_PinHeader_2.54mm:PinHeader_1x03_P2.54mm_Vertical -> TerminalBlock_RND:TerminalBlock_RND_205-00013_1x03_P5.00mm_Horizontal
- J2: value JTAG -> Screw_Terminal_01x03; footprint Connector_PinHeader_2.54mm:PinHeader_2x07_P2.54mm_Vertical -> TerminalBlock_RND:TerminalBlock_RND_205-00013_1x03_P5.00mm_Horizontal
- J3: value BSL_SEL -> USB_B; footprint Connector_PinHeader_2.54mm:PinHeader_1x03_P2.54mm_Vertical -> Connector_USB:USB_B_Lumberg_2411_02_Horizontal
- J4: value USB_B -> Screw_Terminal_01x03; footprint Connector_USB:USB_B_Lumberg_2411_02_Horizontal -> TerminalBlock_RND:TerminalBlock_RND_205-00013_1x03_P5.00mm_Horizontal
- J7: value IR_MOD1 -> JTAG; footprint Connector_PinHeader_2.54mm:PinHeader_1x03_P2.54mm_Vertical -> Connector_IDC:IDC-Header_2x07_P2.54mm_Vertical
- J8: value IR_MOD1 -> BSL_SEL
- L1: footprint Inductor_SMD_Handsoldering_AKL:L_7.3x7.3_H4.5 -> Inductor_THT_AKL:L_Radial_D7.0mm_P3.00mm
- R1: value 93k1 -> 10k
- R10, R36: value 10k -> 470R
- R11, R16, R48: value 330R -> 10k
- R12: value 330R -> 470R
- R13, R14: value 330R -> 27R
- R15: value 330R -> 4k7
- R2: value 30k1 -> 470R
- R20, R37: value 470R -> 470k
- R23, R26: value 18R -> 10k; footprint Resistor_SMD_AKL:R_1206_3216Metric_Pad1.42x1.75mm_HandSolder -> Resistor_SMD_AKL:R_0603_1608Metric_Pad1.05x0.95mm_HandSolder
- R24, R25, R42: value 18R -> 470R; footprint Resistor_SMD_AKL:R_1206_3216Metric_Pad1.42x1.75mm_HandSolder -> Resistor_SMD_AKL:R_0603_1608Metric_Pad1.05x0.95mm_HandSolder
- R27, R28, R43: value 470k -> 470R
- R3: value 27R -> 93k1; footprint Resistor_SMD_AKL:R_0603_1608Metric_Pad1.05x0.95mm_HandSolder -> Resistor_SMD_AKL:R_1206_3216Metric_Pad1.42x1.75mm_HandSolder
- R30: value 470k -> 18R; footprint Resistor_SMD_AKL:R_0603_1608Metric_Pad1.05x0.95mm_HandSolder -> Resistor_SMD_AKL:R_1206_3216Metric_Pad1.42x1.75mm_HandSolder
- R31: value 470k -> 47k
- R33: value 10k -> 330R
- R38, R45, R47: value 10k -> 18R; footprint Resistor_SMD_AKL:R_0603_1608Metric_Pad1.05x0.95mm_HandSolder -> Resistor_SMD_AKL:R_1206_3216Metric_Pad1.42x1.75mm_HandSolder
- R4: value 27R -> 470R
- R44, R46: value 330R -> 470k
- R5: value 47k -> 470R
- R6: value 330R -> 30k1; footprint Resistor_SMD_AKL:R_0603_1608Metric_Pad1.05x0.95mm_HandSolder -> Resistor_SMD_AKL:R_1206_3216Metric_Pad1.42x1.75mm_HandSolder
- R9: value 4k7 -> 18R; footprint Resistor_SMD_AKL:R_0603_1608Metric_Pad1.05x0.95mm_HandSolder -> Resistor_SMD_AKL:R_1206_3216Metric_Pad1.42x1.75mm_HandSolder
- U1: footprint Package_SO_AKL:SOIC-8-1EP_3.9x4.9mm_P1.27mm_EP2.514x3.2mm -> Package_TO_SOT_SMD:TSOT-23-6_HandSoldering
- U2: value FT231XS -> LM324A; footprint Package_SO:SSOP-20_3.9x8.7mm_P0.635mm -> Package_SO_AKL:SOIC-14_3.9x8.7mm_P1.27mm
- U3: value MSP430G2553IPW28 -> FT231XS; footprint Package_SO:TSSOP-28_4.4x9.7mm_P0.65mm -> Package_SO:SSOP-20_3.9x8.7mm_P0.635mm
- U5: value LM324A -> MSP430G2553IPW28; footprint Package_SO_AKL:SOIC-14_3.9x8.7mm_P1.27mm -> Package_SO:TSSOP-28_4.4x9.7mm_P0.65mm
- Y1: moved to B.Cu
- moved J10 163.4 mm to (234.0, 81.2), turned to 180 degrees
- moved R41 161.1 mm to (232.5, 63.0), turned to 90 degrees
- moved U4 155.9 mm to (227.7, 66.4), turned to 90 degrees
- moved J11 153.1 mm to (224.0, 53.8)
- moved C13 152.6 mm to (232.0, 66.8), turned to -90 degrees
- moved R48 150.6 mm to (231.8, 71.5)
- moved R43 148.7 mm to (230.5, 59.9), turned to -90 degrees
- moved R42 143.8 mm to (224.5, 72.5), turned to 90 degrees
- moved Q6 142.8 mm to (235.6, 63.1)
- moved R44 141.5 mm to (227.5, 71.5), turned to 180 degrees
- moved R47 141.4 mm to (235.1, 59.6), turned to 180 degrees
- moved R45 139.5 mm to (219.7, 72.8)
- moved C23 137.5 mm to (223.8, 60.5), turned to 90 degrees
- moved Q5 134.3 mm to (219.1, 69.5), turned to 180 degrees
- moved J9 132.4 mm to (211.0, 81.2), turned to 180 degrees
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Connections:
- C1 pad 2: GND -> Net-(C1-Pad2)
- C10 pad 1: +3V3 -> /3V3OUT
- C11 pad 1: +3V3 -> Net-(C11-Pad1)
- C11 pad 2: GND -> /MODULE2_IN
- C13 pad 1: /USB_D- -> +3V3
- C14 pad 1: /USB_D+ -> +3V3
- C15 pad 1: /FT231_DTR# -> +3V3
- C18 pad 1: Net-(C18-Pad1) -> +3V3
- C18 pad 2: /MODULE5_IN -> GND
- C19 pad 2: /MODULE1_IN -> /MODULE3_IN
- C2 pad 1: Net-(C1-Pad1) -> +3V3
- C2 pad 2: GND -> Net-(C2-Pad2)
- C20 pad 1: Net-(C20-Pad1) -> /FT231_DTR#
- C20 pad 2: /MODULE2_IN -> GND
- C21 pad 2: /MODULE3_IN -> /MODULE4_IN
- C22 pad 2: /MODULE4_IN -> /MODULE6_IN
- C23 pad 2: /MODULE6_IN -> /MODULE5_IN
- C3 pad 1: Net-(C3-Pad1) -> +3V3
- C3 pad 2: Net-(C3-Pad2) -> GND
- C4 pad 2: Net-(C4-Pad2) -> GND
- C5 pad 1: +3V3 -> Net-(C6-Pad1)
- C6 pad 1: +3V3 -> Net-(C6-Pad1)
- C7 pad 1: +3V3 -> Net-(C7-Pad1)
- C7 pad 2: GND -> /MODULE1_IN
- C8 pad 1: /3V3OUT -> /USB_D-
- C9 pad 1: +3V3 -> /USB_D+
- D1 pad 1: Net-(C1-Pad1) -> GND
- D1 pad 2: GND -> Net-(D1-Pad2)
- D10 pad 1: GND -> /RX_LED
- D2 pad 1: Net-(D2-Pad1) -> Net-(C6-Pad1)
- D2 pad 2: Net-(D2-Pad2) -> GND
- J1 pad 1: Net-(D1-Pad3) -> Net-(D2-Pad3)
- J1 pad 2: Net-(D1-Pad4) -> Net-(D2-Pad4)
- J2 pad 1: /FT231_DTR# -> Net-(J2-Pad1)
- J2 pad 2: unconnected-(J2-Pad2) -> GND
- J2 pad 3: unconnected-(J2-Pad3) -> Net-(J2-Pad3)
- J3 pad 1: /MSP_UART_TX -> Net-(J3-Pad1)
- J3 pad 2: /FT231_RX -> /USB_D-
- J3 pad 3: /MSP_BSL_TX -> /USB_D+
- J4 pad 2: /USB_D- -> GND
- J4 pad 3: /USB_D+ -> Net-(J4-Pad3)
- J7 pad 1: Net-(J7-Pad1) -> /FT231_DTR#
- J7 pad 2: GND -> unconnected-(J7-Pad2)
- J7 pad 3: Net-(J7-Pad3) -> unconnected-(J7-Pad3)
- J8 pad 1: Net-(J8-Pad1) -> /MSP_UART_TX
- J8 pad 2: GND -> /FT231_RX
- J8 pad 3: Net-(J8-Pad3) -> /MODULE1_IN
- L1 pad 1: Net-(C3-Pad2) -> Net-(C1-Pad2)
- R1 pad 2: Net-(C4-Pad2) -> Net-(Q1-Pad1)
- R10 pad 1: GND -> Net-(D5-Pad2)
- R10 pad 2: /VUSB_SENSE -> /MODULE3_STATUS
- R11 pad 1: /FT231_RTS# -> GND
- R11 pad 2: /TCK -> /MODULE1_IN
- R12 pad 1: Net-(D3-Pad2) -> Net-(D6-Pad2)
- R12 pad 2: /MODULE1_STATUS -> /MODULE4_STATUS
- R13 pad 1: Net-(D4-Pad2) -> /USB_D-
- R13 pad 2: /MODULE2_STATUS -> /FT_USB-
- R14 pad 1: Net-(D5-Pad2) -> /USB_D+
- R14 pad 2: /MODULE3_STATUS -> /FT_USB+
- R15 pad 1: Net-(D6-Pad2) -> Net-(J3-Pad1)
- R15 pad 2: /MODULE4_STATUS -> /VUSB_SENSE
- R16 pad 1: Net-(D7-Pad2) -> +3V3
- R16 pad 2: /MODULE5_STATUS -> Net-(Q2-Pad1)
- R17 pad 1: /MODULE5_OUT -> Net-(D7-Pad2)
- R17 pad 2: Net-(Q1-Pad1) -> /MODULE5_STATUS
- R18 pad 1: +3V3 -> GND
- R18 pad 2: Net-(Q2-Pad1) -> /VUSB_SENSE
- R19 pad 1: /MODULE1_OUT -> /MODULE2_OUT
- R2 pad 1: Net-(C4-Pad2) -> Net-(D1-Pad2)
- R2 pad 2: GND -> /MODULE1_STATUS
- R20 pad 1: /MODULE2_OUT -> Net-(J4-Pad1)
- R20 pad 2: Net-(Q3-Pad1) -> Net-(C11-Pad1)
- R21 pad 1: /MODULE3_OUT -> Net-(D8-Pad2)
- R21 pad 2: Net-(Q4-Pad1) -> /MODULE6_STATUS
- R22 pad 1: Net-(Q1-Pad3) -> Net-(Q2-Pad3)
- R22 pad 2: Net-(J6-Pad3) -> Net-(J4-Pad3)
- R23 pad 1: Net-(Q2-Pad3) -> GND
- R23 pad 2: Net-(J7-Pad3) -> /MODULE2_IN
- R24 pad 1: Net-(Q3-Pad3) -> Net-(D9-Pad2)
- R24 pad 2: Net-(J8-Pad3) -> /GP_LED
- R25 pad 1: Net-(Q4-Pad3) -> Net-(D10-Pad2)
- R25 pad 2: Net-(J9-Pad3) -> +3V3
- R26 pad 1: Net-(Q5-Pad3) -> +3V3
- R26 pad 2: Net-(J10-Pad3) -> Net-(Q3-Pad1)
- R27 pad 1: Net-(J6-Pad1) -> /MODULE3_OUT
- R27 pad 2: Net-(C18-Pad1) -> Net-(Q3-Pad1)
- R28 pad 1: Net-(J7-Pad1) -> Net-(D11-Pad2)
- R28 pad 2: Net-(C19-Pad1) -> +3V3
- R29 pad 1: Net-(J8-Pad1) -> Net-(J6-Pad1)
- R29 pad 2: Net-(C20-Pad1) -> Net-(C19-Pad1)
- R3 pad 1: /USB_D- -> +3V3
- R3 pad 2: Net-(R3-Pad2) -> Net-(C2-Pad2)
- R30 pad 1: Net-(J9-Pad1) -> Net-(Q3-Pad3)
- R30 pad 2: Net-(C21-Pad1) -> Net-(J6-Pad3)
- R31 pad 1: Net-(J10-Pad1) -> +3V3
- R31 pad 2: Net-(C22-Pad1) -> /FT231_DTR#
- R32 pad 2: /MODULE5_IN -> /MODULE3_IN
- R33 pad 1: GND -> /FT231_RTS#
- R33 pad 2: /MODULE1_IN -> /TCK
- R34 pad 1: GND -> +3V3
- R34 pad 2: /MODULE2_IN -> /GP_BUTTON
- R35 pad 1: GND -> +3V3
- R35 pad 2: /MODULE3_IN -> Net-(Q4-Pad1)
- R36 pad 1: GND -> /MODULE4_OUT
- R36 pad 2: /MODULE4_IN -> Net-(Q4-Pad1)
- R37 pad 1: /MODULE4_OUT -> Net-(J9-Pad1)
- R37 pad 2: Net-(Q5-Pad1) -> Net-(C21-Pad1)
- R38 pad 1: +3V3 -> Net-(Q4-Pad3)
- R38 pad 2: Net-(Q1-Pad1) -> Net-(J9-Pad3)
- R39 pad 1: +3V3 -> GND
- R39 pad 2: Net-(Q3-Pad1) -> /MODULE4_IN
- R4 pad 1: /USB_D+ -> +3V3
- R4 pad 2: Net-(R4-Pad2) -> Net-(D3-Pad2)
- R40 pad 2: Net-(Q4-Pad1) -> Net-(Q5-Pad1)
- R41 pad 2: Net-(Q5-Pad1) -> Net-(Q6-Pad1)
- R42 pad 1: Net-(Q6-Pad3) -> /MODULE6_OUT
- R42 pad 2: Net-(J11-Pad3) -> Net-(Q5-Pad1)
- R43 pad 1: Net-(J11-Pad1) -> /MODULE5_OUT
- R43 pad 2: Net-(C23-Pad1) -> Net-(Q6-Pad1)
- R44 pad 1: Net-(D8-Pad2) -> Net-(J10-Pad1)
- R44 pad 2: /MODULE6_STATUS -> Net-(C22-Pad1)
- R45 pad 1: GND -> Net-(Q5-Pad3)
- R45 pad 2: /MODULE6_IN -> Net-(J10-Pad3)
- R46 pad 1: +3V3 -> Net-(J11-Pad1)
- R46 pad 2: Net-(D9-Pad2) -> Net-(C23-Pad1)
- R47 pad 1: +3V3 -> Net-(Q6-Pad3)
- R47 pad 2: /GP_BUTTON -> Net-(J11-Pad3)
- R48 pad 1: Net-(D10-Pad2) -> GND
- R48 pad 2: /GP_LED -> /MODULE6_IN
- R5 pad 1: +3V3 -> /MODULE1_OUT
- R5 pad 2: /FT231_DTR# -> Net-(Q1-Pad1)
- R6 pad 1: Net-(D2-Pad2) -> Net-(C2-Pad2)
- R6 pad 2: +3V3 -> GND
- R9 pad 1: Net-(J4-Pad1) -> Net-(Q1-Pad3)
- R9 pad 2: /VUSB_SENSE -> Net-(J2-Pad3)
- U1 pad 1: Net-(C4-Pad2) -> Net-(C2-Pad2)
- U1 pad 2: Net-(C1-Pad1) -> Net-(C6-Pad1)
- U1 pad 3: Net-(C1-Pad1) -> Net-(C6-Pad1)
- U1 pad 5: Net-(C3-Pad2) -> Net-(C1-Pad2)
- U1 pad 6: Net-(C3-Pad1) -> Net-(C1-Pad1)
- U2 pad 1: /FT231_DTR# -> Net-(C7-Pad1)
- U2 pad 10: /VUSB_SENSE -> Net-(J9-Pad1)
- U2 pad 11: Net-(R4-Pad2) -> GND
- U2 pad 12: Net-(R3-Pad2) -> Net-(J6-Pad1)
- U2 pad 13: /3V3OUT -> GND
- U2 pad 14: /3V3OUT -> Net-(C19-Pad1)
- U2 pad 2: /FT231_RTS# -> GND
- U2 pad 3: /3V3OUT -> Net-(J2-Pad1)
- U2 pad 4: /FT231_RX -> +3V3
- U2 pad 5: unconnected-(U2-Pad5) -> Net-(J4-Pad1)
- U2 pad 7: unconnected-(U2-Pad7) -> Net-(C11-Pad1)
- U2 pad 8: unconnected-(U2-Pad8) -> Net-(C21-Pad1)
- U2 pad 9: unconnected-(U2-Pad9) -> GND
- U3 pad 1: +3V3 -> /FT231_DTR#
- U3 pad 10: /MODULE1_OUT -> unconnected-(U3-Pad10)
- U3 pad 11: /MODULE2_OUT -> /FT_USB+
- U3 pad 12: /MODULE3_OUT -> /FT_USB-
- U3 pad 13: /MODULE3_STATUS -> /3V3OUT
- U3 pad 14: /MODULE4_STATUS -> /3V3OUT
- U3 pad 15: /MODULE5_STATUS -> +3V3
- U3 pad 16: /MODULE4_OUT -> GND
- U3 pad 17: /MODULE5_OUT -> /TX_LED
- U3 pad 18: /MODULE6_OUT -> /RX_LED
- U3 pad 19: /MODULE6_STATUS -> /VUSB_SENSE
- U3 pad 2: /MODULE6_IN -> /FT231_RTS#
- U3 pad 20: /GP_LED -> /FT231_TX
- U3 pad 3: /FT231_TX -> /3V3OUT
- U3 pad 4: /MSP_UART_TX -> /FT231_RX
- U3 pad 5: /MODULE1_IN -> unconnected-(U3-Pad5)
- U3 pad 6: /MODULE2_IN -> GND
- U3 pad 7: /MODULE3_IN -> unconnected-(U3-Pad7)
- U3 pad 8: /MODULE2_STATUS -> unconnected-(U3-Pad8)
- U3 pad 9: /MODULE1_STATUS -> unconnected-(U3-Pad9)
- U4 pad 1: Net-(C18-Pad1) -> Net-(C22-Pad1)
- U4 pad 3: Net-(J6-Pad1) -> Net-(J10-Pad1)
- U5 pad 1: Net-(C19-Pad1) -> +3V3
- U5 pad 10: Net-(J9-Pad1) -> /MODULE2_STATUS
- U5 pad 11: GND -> /MODULE1_STATUS
- U5 pad 12: Net-(J10-Pad1) -> /MODULE6_OUT
- U5 pad 13: GND -> /MODULE4_OUT
- U5 pad 14: Net-(C22-Pad1) -> /MODULE2_OUT
- U5 pad 2: GND -> /MODULE4_IN
- U5 pad 3: Net-(J7-Pad1) -> /FT231_TX
- U5 pad 4: +3V3 -> /MSP_UART_TX
- U5 pad 5: Net-(J8-Pad1) -> /MODULE2_IN
- U5 pad 6: GND -> /MODULE3_IN
- U5 pad 7: Net-(C20-Pad1) -> /MODULE1_IN
- U5 pad 8: Net-(C21-Pad1) -> /MODULE4_STATUS
- U5 pad 9: GND -> /MODULE3_STATUS
- Y1 pad 1: Net-(U3-Pad26) -> Net-(U5-Pad26)
- Y1 pad 2: Net-(U3-Pad27) -> Net-(U5-Pad27)
Routing:
- net +3V3: track 0.00 -> 198.1 mm, vias 0 -> 10
- net /MODULE6_IN: track 0.00 -> 106.1 mm, vias 0 -> 2
- net /MODULE6_OUT: track 0.00 -> 94.2 mm
- net /MODULE5_IN: track 0.00 -> 88.9 mm
- net /MODULE5_OUT: track 0.00 -> 87.2 mm, vias 0 -> 2
- net /MODULE4_OUT: track 0.00 -> 80.7 mm
- net /FT231_DTR#: track 0.00 -> 62.0 mm, vias 0 -> 2
- net /MODULE1_IN: track 0.00 -> 62.0 mm
- net /MODULE2_OUT: track 0.00 -> 56.4 mm
- net /FT231_RTS#: track 0.00 -> 56.0 mm, vias 0 -> 4
- net /MODULE3_OUT: track 0.00 -> 54.3 mm, vias 0 -> 2
- net /FT231_TX: track 0.00 -> 53.7 mm
- net /MODULE1_OUT: track 0.00 -> 34.5 mm, vias 0 -> 2
- net /MSP_UART_TX: track 0.00 -> 33.6 mm
- net /MODULE4_IN: track 0.00 -> 33.5 mm, vias 0 -> 2
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- added copper zone on B.Cu, net GND
- added copper zone on F.Cu, net GND
Other:
- board outline added: 160 x 35 mm

Commit message: finished board
Parts:
- added REF**: OSHW-Logo2_9.8x8mm_SilkScreen, Symbol:OSHW-Logo2_9.8x8mm_SilkScreen, F.Cu at (169.0, 80.2)
- moved L1 0.35 mm to (127.7, 55.4)
- moved C14 0.25 mm to (137.0, 64.2)
- moved R33 0.15 mm to (133.4, 58.8)
Routing:
- net +3V3: track 198.1 -> 238.4 mm, vias 10 -> 12
- net /3V3OUT: track 3.77 -> 11.8 mm, vias 0 -> 2
- net GND: track 15.5 -> 8.67 mm, vias 11 -> 94
- net Net-(C1-Pad2): track 4.68 -> 8.58 mm
Other:
- board text added: "BSL"
- board text added: "UART"

Commit message: finished hardware revision 1.0
Parts:
- added REF**: MountingHole_3.2mm_M3_DIN965, MountingHole:MountingHole_3.2mm_M3_DIN965, F.Cu at (167.0, 81.2)
- U2: renamed from U4; footprint Package_SO_AKL:SOIC-8-1EP_3.9x4.9mm_P1.27mm_EP2.514x3.2mm -> Package_SO_AKL:SOIC-8_3.9x4.9mm_P1.27mm
- Y1: moved to F.Cu
- moved REF** 25.5 mm to (194.5, 80.5)
- moved Y1 1.90 mm to (139.5, 67.8), turned to -90 degrees
- renumbered C5 to C1, C20 to C10, C1 to C11, C2 to C12, C22 to C13, C10 to C14, C3 to C15, C4 to C16, C12 to C17, C23 to C18, C13 to C19, C8 to C2, C7 to C20, C11 to C21, C19 to C22, C21 to C23, C14 to C3, C6 to C4, C16 to C5, C15 to C6, C9 to C7, C17 to C8, C18 to C9, D2 to D1, D8 to D10, D9 to D11, D10 to D2, D11 to D3, D3 to D4, D1 to D5, D4 to D6, D5 to D7, D6 to D8, D7 to D9, J6 to J10, J9 to J11, J7 to J2, J8 to J3, J10 to J4, J3 to J5, J11 to J6, J5 to J7, J2 to J8, J4 to J9, Q5 to Q1, Q6 to Q2, Q1 to Q3, Q2 to Q4, Q3 to Q5, Q4 to Q6, R42 to R1, R48 to R10, R25 to R11, R28 to R12, R4 to R13, R15 to R14, R18 to R15, R33 to R16, R43 to R17, R41 to R18, R47 to R19, R40 to R2, R46 to R20, R49 to R21, R34 to R22, R2 to R23, R7 to R24, R10 to R25, R12 to R26, R17 to R27, R21 to R28, R24 to R29, R13 to R3, R5 to R30, R19 to R31, R27 to R32, R36 to R33, R1 to R34, R16 to R35, R26 to R36, R35 to R37, R9 to R38, R22 to R39, R14 to R4, R30 to R40, R38 to R41, R8 to R42, R20 to R43, R29 to R44, R37 to R45, R11 to R46, R23 to R47, R32 to R48, R39 to R49, R45 to R5, R31 to R6, R44 to R7, R3 to R8, R6 to R9, TP5 to TP10, TP3 to TP2, TP6 to TP3, TP7 to TP4, TP8 to TP5, TP9 to TP6, TP10 to TP7, TP2 to TP8, TP4 to TP9, U5 to U4, U2 to U5
Connections:
- U4 pad 26: Net-(U5-Pad26) -> Net-(U4-Pad26)
- U4 pad 27: Net-(U5-Pad27) -> Net-(U4-Pad27)
- Y1 pad 1: Net-(U5-Pad26) -> Net-(U4-Pad27)
- Y1 pad 2: Net-(U5-Pad27) -> Net-(U4-Pad26)
Routing:
- net Net-(U5-Pad26): track 10.5 -> 0.00 mm, vias 1 -> 0
- net Net-(U4-Pad26): track 0.00 -> 10.5 mm, vias 0 -> 1
- net Net-(U5-Pad27): track 8.65 -> 0.00 mm, vias 1 -> 0
- net Net-(U4-Pad27): track 0.00 -> 8.65 mm, vias 0 -> 1
- net /MODULE5_OUT: track 87.2 -> 93.6 mm
- net /FT231_RTS#: track 55.5 -> 60.8 mm, vias 4 -> 8
- net +3V3: track 238.4 -> 240.2 mm
- net Net-(J4-Pad3): track 10.1 -> 9.51 mm
- net /FT231_DTR#: vias 2 -> 6
- net GND: vias 94 -> 103
Other:
- board text added: "RX"
- board text added: "TX"

Commit message: production hw rev 1.0
Parts:
- C2, C7: footprint Capacitor_SMD_Handsoldering_AKL:C_0805_2012Metric -> Capacitor_SMD_Handsoldering_AKL:C_0603_1608Metric_Pad1.08x0.95mm
- R16: footprint Resistor_SMD_AKL:R_0603_1608Metric_Pad1.05x0.95mm_HandSolder -> Resistor_SMD_AKL:R_0805_2012Metric_Pad1.20x1.40mm_HandSolder
- moved REF** 27.3 mm to (214.8, 62.2)
- moved H2 2.30 mm to (217.6, 81.8)
- moved REF** 1.69 mm to (168.6, 81.8)
- moved R16 0.20 mm to (133.6, 58.8)
- moved H3 0.11 mm to (168.6, 55.2)
- turned D5 to 180 degrees
- turned D6 to 180 degrees
Routing:
- net Net-(D6-Pad2): track 2.00 -> 2.72 mm
- net Net-(D5-Pad2): track 2.00 -> 2.72 mm
- net GND: vias 103 -> 104
Other:
- board text added: "3V3"
- board text added: "DTR"
- board text added: "GND"
- board text added: "In"
- board text added: "Infrared model train detection Hardware Rev. 1.0"
- board text added: "Out"
- board text added: "RTS"

Commit message: finished hardware rev 1.1
Parts:
- removed the REF** at (168.6, 81.8)
- removed the REF** at (214.8, 62.2)
- added 3V3: TestPoint, TestPoint:TestPoint_Pad_D1.5mm, F.Cu at (170.0, 82.8)
- added GND: TestPoint, TestPoint:TestPoint_Pad_D1.5mm, F.Cu at (130.2, 75.0)
- added JP1: Jumper_2_Open, 4ms_SolderJumper:JUMPER_SMD_1x2, B.Cu at (163.2, 74.8)
- added R50: 470k, Resistor_SMD_AKL:R_0603_1608Metric_Pad1.05x0.95mm_HandSolder, F.Cu at (187.8, 70.0)
- added REF**: OSHW-Logo2_7.3x6mm_SilkScreen, Symbol:OSHW-Logo2_7.3x6mm_SilkScreen, F.Cu at (214.8, 62.0)
- added SW2: SW_Push, Button_Switch_THT:SW_PUSH_6mm, F.Cu at (117.2, 65.2)
- added TP11: TestPoint, TestPoint:TestPoint_Pad_1.5x1.5mm, F.Cu at (177.2, 68.5)
- C10: value 2n2 -> 1n
- C2, C7: footprint Capacitor_SMD_Handsoldering_AKL:C_0603_1608Metric_Pad1.08x0.95mm -> Capacitor_SMD_Handsoldering_AKL:C_0805_2012Metric
- J3: footprint Connector_PinHeader_2.54mm:PinHeader_1x03_P2.54mm_Vertical -> Connector_PinHeader_2.54mm:PinHeader_2x03_P2.54mm_Vertical
- J7: value Screw_Terminal_01x07 -> Screw_Terminal_01x08; footprint TerminalBlock_RND:TerminalBlock_RND_205-00006_1x07_P5.00mm_Horizontal -> TerminalBlock_RND:TerminalBlock_RND_205-00007_1x08_P5.00mm_Horizontal
- R16: value 330R -> 10k; footprint Resistor_SMD_AKL:R_0805_2012Metric_Pad1.20x1.40mm_HandSolder -> Resistor_SMD_AKL:R_0603_1608Metric_Pad1.05x0.95mm_HandSolder
- R45: value 470k -> 10k
- moved R45 81.6 mm to (119.2, 73.8), turned to 0 degrees
- moved J2 15.7 mm to (156.8, 53.7), turned to -90 degrees
- moved R43 13.8 mm to (200.8, 65.5), turned to 90 degrees
- moved TP4 11.7 mm to (114.5, 72.8)
- moved R16 10.3 mm to (128.2, 67.5), turned to 0 degrees
- moved J7 5.10 mm to (164.5, 81.0)
- moved R44 4.25 mm to (200.8, 69.8), turned to -90 degrees
- moved R20 1.52 mm to (227.5, 59.8)
- moved D5 1.41 mm to (160.5, 74.8), turned to 90 degrees
- moved D6 1.41 mm to (155.5, 74.8), turned to 90 degrees
- moved D7 1.41 mm to (150.5, 74.8), turned to 90 degrees
- moved D8 1.41 mm to (145.5, 74.8), turned to 90 degrees
- moved D9 1.41 mm to (140.5, 74.8), turned to 90 degrees
- moved R28 1.41 mm to (133.8, 74.8), turned to 90 degrees
- moved D10 1.25 mm to (135.5, 74.8), turned to 90 degrees
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Connections:
- C10 pad 1: /FT231_DTR# -> /TDO/TDI
- C14 pad 1: /3V3OUT -> +3V3
- D10 pad 1: GND -> Net-(D10-K)
- D5 pad 1: GND -> Net-(D10-K)
- D6 pad 1: GND -> Net-(D10-K)
- D7 pad 1: GND -> Net-(D10-K)
- D8 pad 1: GND -> Net-(D10-K)
- D9 pad 1: GND -> Net-(D10-K)
- J10 pad 1: Net-(J10-Pad1) -> Net-(J10-Pin_1)
- J11 pad 1: Net-(J11-Pad1) -> Net-(J11-Pin_1)
- J2 pad 1: /FT231_DTR# -> /TDO/TDI
- J2 pad 8: /FT231_RTS# -> unconnected-(J2-Pin_8-Pad8)
- J3 pad 2: /FT231_RX -> /MSP_UART_RX
- J3 pad 3: /MODULE1_IN -> /FT231_RX
- J4 pad 1: Net-(J4-Pad1) -> Net-(J4-Pin_1)
- J6 pad 1: Net-(J6-Pad1) -> Net-(J6-Pin_1)
- J7 pad 1: /MODULE1_STATUS -> +3V3
- J7 pad 2: /MODULE2_STATUS -> /MODULE1_STATUS
- J7 pad 3: /MODULE3_STATUS -> /MODULE2_STATUS
- J7 pad 4: /MODULE4_STATUS -> /MODULE3_STATUS
- J7 pad 5: /MODULE5_STATUS -> /MODULE4_STATUS
- J7 pad 6: /MODULE6_STATUS -> /MODULE5_STATUS
- J7 pad 7: GND -> /MODULE6_STATUS
- J8 pad 1: Net-(J8-Pad1) -> Net-(J8-Pin_1)
- J9 pad 1: Net-(J9-Pad1) -> Net-(J9-Pin_1)
- R20 pad 1: Net-(J6-Pad1) -> Net-(J6-Pin_1)
- R42 pad 1: Net-(J8-Pad1) -> Net-(J8-Pin_1)
- R43 pad 1: Net-(J9-Pad1) -> Net-(J10-Pin_1)
- R43 pad 2: Net-(C21-Pad1) -> Net-(C22-Pad1)
- R44 pad 1: Net-(J10-Pad1) -> Net-(J11-Pin_1)
- R44 pad 2: Net-(C22-Pad1) -> Net-(C23-Pad1)
- R45 pad 1: Net-(J11-Pad1) -> /FT231_DTR#
- R45 pad 2: Net-(C23-Pad1) -> /TDO/TDI
- R6 pad 2: /FT231_DTR# -> /TDO/TDI
- R7 pad 1: Net-(J4-Pad1) -> Net-(J4-Pin_1)
- U2 pad 2: GND -> Net-(J4-Pin_1)
- U2 pad 3: Net-(J4-Pad1) -> GND
- U2 pad 5: Net-(J6-Pad1) -> GND
- U2 pad 6: GND -> Net-(J6-Pin_1)
- U3 pad 13: /3V3OUT -> +3V3
- U3 pad 14: /3V3OUT -> +3V3
- U3 pad 3: /3V3OUT -> +3V3
- U4 pad 10: /MODULE2_STATUS -> /MODULE1_STATUS
- U4 pad 11: /MODULE1_STATUS -> /MODULE1_OUT
- U4 pad 16: /MODULE1_OUT -> /MODULE4_STATUS
- U4 pad 17: /MODULE5_OUT -> /MODULE3_OUT
- U4 pad 18: /MODULE3_OUT -> /MODULE5_OUT
- U4 pad 24: /FT231_DTR# -> /TDO/TDI
- U4 pad 25: /FT231_RTS# -> /TCK
- U4 pad 3: /FT231_TX -> /MSP_UART_RX
- U4 pad 8: /MODULE4_STATUS -> /MODULE3_STATUS
- U4 pad 9: /MODULE3_STATUS -> /MODULE2_STATUS
- U5 pad 10: Net-(J11-Pad1) -> GND
- U5 pad 12: Net-(J10-Pad1) -> GND
- U5 pad 13: GND -> Net-(J10-Pin_1)
- U5 pad 2: GND -> Net-(J8-Pin_1)
- U5 pad 3: Net-(J8-Pad1) -> GND
- U5 pad 5: Net-(J9-Pad1) -> GND
- U5 pad 6: GND -> Net-(J9-Pin_1)
- U5 pad 9: GND -> Net-(J11-Pin_1)
Routing:
- net +3V3: track 240.2 -> 319.6 mm
- net /TDO/TDI: track 0.00 -> 68.7 mm, vias 0 -> 2
- net /FT231_DTR#: track 62.0 -> 10.4 mm, vias 6 -> 0
- net /FT231_RTS#: track 60.6 -> 23.2 mm, vias 8 -> 0
- net /MSP_UART_RX: track 0.00 -> 37.0 mm
- net /FT231_TX: track 53.7 -> 19.1 mm
- net Net-(D10-K): track 0.00 -> 33.0 mm, vias 0 -> 6
- net Net-(J11-Pin_1): track 0.00 -> 23.0 mm
- net Net-(J8-Pin_1): track 0.00 -> 22.5 mm, vias 0 -> 1
- net Net-(J8-Pad1): track 22.1 -> 0.00 mm, vias 1 -> 0
- net Net-(J11-Pad1): track 21.0 -> 0.00 mm
- net Net-(J9-Pad1): track 20.2 -> 0.00 mm, vias 2 -> 0
- net Net-(J10-Pin_1): track 0.00 -> 17.6 mm
- net Net-(J10-Pad1): track 17.5 -> 0.00 mm, vias 1 -> 0
- net Net-(J9-Pin_1): track 0.00 -> 16.3 mm, vias 0 -> 2
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Other:
- board text added: "Infrared model train detection Hardware Rev. 1.1"
- board text removed: "Infrared model train detection Hardware Rev. 1.0"
