File: board/ir-train-detector.kicad_sch (KiCad schematic)
At the start: 91 parts, among them J1 ST_01x02, J10 IR_MOD1, J2 JTAG, J3 BSL_SEL, J4 USB_B, J5 Conn_01x07, J6 IR_MOD1, J7 IR_MOD1, J8 IR_MOD1, J9 IR_MOD1, Q1 AO3407A, Q2 AO3407A, Q3 AO3407A, Q4 AO3407A, Q5 AO3407A, U1 AP63300WU, U2 FT231XS, U3 MSP430G2553IPW28, U4 LM358, U5 LM324A

Commit message: finished schematic
Parts:
- removed J10, J6, J7, J8, J9: IR_MOD1, symbol Connector_Generic:Conn_01x03
- removed J5: Conn_01x07, symbol Connector_Generic:Conn_01x07
- added C23: 33n, Capacitor_SMD_Handsoldering_AKL:C_0603_1608Metric, symbol Device:C_Small
- added D10, D8: LED, LED_SMD:LED_0603_1608Metric_Pad1.05x0.95mm_HandSolder, symbol Device:LED
- added D11: LED, symbol Device:LED
- added D9: LED_PWR, LED_SMD:LED_0603_1608Metric_Pad1.05x0.95mm_HandSolder, symbol Device:LED
- added J10, J11, J12, J6, J8, J9: Screw_Terminal_01x03, TerminalBlock_RND:TerminalBlock_RND_205-00013_1x03_P5.00mm_Horizontal, symbol Connector:Screw_Terminal_01x03
- added J7: Screw_Terminal_01x08, symbol Connector:Screw_Terminal_01x08
- added Q6: AO3407A, Package_TO_SOT_SMD_AKL:SOT-23, symbol Transistor_MOSFET_AKL:AO3407A
- added R42: 18R, Resistor_SMD_AKL:R_1206_3216Metric_Pad1.42x1.75mm_HandSolder, symbol Device:R_Small
- added R43: 470k, Resistor_SMD_AKL:R_0603_1608Metric_Pad1.05x0.95mm_HandSolder, symbol Device:R_Small
- added R44, R46, R48: 470R, Resistor_SMD_AKL:R_0603_1608Metric_Pad1.05x0.95mm_HandSolder, symbol Device:R_Small
- added R45, R47, R49: 10k, Resistor_SMD_AKL:R_0603_1608Metric_Pad1.05x0.95mm_HandSolder, symbol Device:R_Small
- added SW1: SW_Push, Button_Switch_THT:SW_PUSH_6mm, symbol Switch:SW_Push
- added TP1, TP11, TP12, TP13, TP14, TP15, TP16, TP17, TP18, TP19, TP2, TP20, TP21, TP3, TP6, TP7, TP8: TestPoint, TestPoint:TestPoint_Pad_D1.5mm, symbol Connector:TestPoint
- added TP10, TP22, TP23, TP24, TP25, TP4, TP5, TP9: TestPoint, symbol Connector:TestPoint
- added Y1: 32768Hz, Crystal:Crystal_C26-LF_D2.1mm_L6.5mm_Horizontal, symbol Device:Crystal
- C1: footprint Capacitor_THT:CP_Radial_D12.5mm_P5.00mm -> Capacitor_THT_AKL:CP_Radial_D12.5mm_P5.00mm
- C12: footprint Capacitor_SMD_Handsoldering_AKL:C_0603_1608Metric -> Capacitor_THT_AKL:CP_Radial_D4.0mm_P1.50mm
- C15, C4: footprint Capacitor_SMD_Handsoldering_AKL:C_0603_1608Metric -> Capacitor_SMD_Handsoldering_AKL:C_0805_2012Metric
- C5, C6: footprint Capacitor_SMD_Handsoldering_AKL:C_0805_2012Metric -> Capacitor_SMD_Handsoldering_AKL:C_1206_3216Metric
- J1, R17, R18, R19, R20, R21, R27, R28, R29, R30, R31, R32, R33, R35, R36, R37, R38, R39, R40, R41: footprint (none) -> Resistor_SMD_AKL:R_0603_1608Metric_Pad1.05x0.95mm_HandSolder
- J2: footprint (none) -> Connector_IDC:IDC-Header_2x07_P2.54mm_Vertical
- J3: footprint (none) -> Connector_PinHeader_2.54mm:PinHeader_1x03_P2.54mm_Vertical
- L1: footprint Inductor_SMD_Handsoldering_AKL:L_7.3x7.3_H4.5 -> Inductor_THT_AKL:L_Radial_D7.0mm_P3.00mm
- R1, R2: footprint Resistor_SMD_AKL:R_0603_1608Metric_Pad1.05x0.95mm_HandSolder -> Resistor_SMD_AKL:R_1206_3216Metric_Pad1.42x1.75mm_HandSolder
- R12, R13, R14, R15, R16, R6: value 330R -> 470R
- R22, R23, R24, R25, R26: footprint (none) -> Resistor_SMD_AKL:R_1206_3216Metric_Pad1.42x1.75mm_HandSolder
- R34, R7: value 10k -> 470R
- U1: footprint (none) -> Package_SO_AKL:SOIC-8-1EP_3.9x4.9mm_P1.27mm_EP2.514x3.2mm
- U4: footprint 4ms_Package_SSOP:TSSOP-8_4.4x3mm_Pitch0.65mm -> Package_SO_AKL:SOIC-8-1EP_3.9x4.9mm_P1.27mm_EP2.514x3.2mm
Connections:
- net +3V3: now also R34.1, R8.1, J7.1 (Pin_1), Q6.2 (S), R46.1, R47.1, TP4.1; no longer R7.1
- net FT231_DTR#: now also TP25.1
- net FT231_RTS#: now also TP24.1
- net FT231_RX: now also TP23.1
- net FT231_TX: now also TP22.1
- net GND: now also U4.6 (-), D10.1 (K), D8.1 (K), D9.1 (K), J10.2 (Pin_2), J11.2 (Pin_2), J12.2 (Pin_2), J6.2 (Pin_2), J7.8 (Pin_8), J8.2 (Pin_2), J9.2 (Pin_2), R45.1, R49.1, SW1.1, TP5.1; no longer R34.1, R8.2
- net MODULE1_IN: now also C20.2, R35.2, TP18.1; no longer C19.2, R33.2
- net MODULE1_STATUS: now also J7.2 (Pin_2)
- net MODULE2_IN: now also C21.2, R36.2, TP19.1; no longer C20.2, R34.2
- net MODULE2_STATUS: now also J7.3 (Pin_3)
- net MODULE3_IN: now also C22.2, R45.2, TP20.1; no longer C21.2, R35.2
- net MODULE3_STATUS: now also J7.4 (Pin_4)
- net MODULE4_IN: now also C23.2, R49.2, TP21.1; no longer C22.2, R36.2
- net MODULE4_STATUS: now also J7.5 (Pin_5)
- net MODULE5_IN: now also TP3.1
- net MODULE5_STATUS: now also J7.6 (Pin_6)
- net at R30.2, U5.8: now also C22.1, TP16.1; no longer C21.1
- net at R28.1, U5.3 (+): now also J9.1 (Pin_1), TP10.1
- net at R28.2, U5.1: now also C20.1, TP14.1; no longer C19.1
- net at R25.2: now also J11.3 (Pin_3)
- net at R30.1, U5.10 (+): now also J11.1 (Pin_1), TP12.1
- net at R27.1, U4.3 (+): now also J8.1 (Pin_1), TP1.1
- net at R22.2: now also J8.3 (Pin_3)
- net at R24.2: now also J10.3 (Pin_3)
- net at R31.1, U5.12 (+): now also J12.1 (Pin_1), TP13.1
- net at R31.2, U5.14: now also C23.1, TP17.1; no longer C22.1
- net at R23.2: now also J9.3 (Pin_3)
- net at C18.1, R27.2, U4.1: now also TP2.1
- net MODULE6_OUT: now reaches U3.18 (TA1.2/P2.5)
- net MODULE6_OUT: now also R7.1
- net MODULE6_STATUS: now reaches U3.19 (P3.5/TA0.1)
- net MODULE6_STATUS: now also J7.7 (Pin_7), R44.2
- net MODULE6_IN: now reaches U3.2 (TA0CLK/ACLK/A0/CA0/P1.0)
- net MODULE6_IN: now also C19.2, R33.2, TP8.1
- net GP_LED: now reaches U3.20 (P3.6/TA0.2)
- net GP_LED: now also D11.1 (K), R48.2
- net GP_BUTTON: now reaches U3.21 (P3.7/TA1CLK/CAOUT)
- net GP_BUTTON: now also R47.2, SW1.2, TP9.1
- net at U3.26 (XOUT/P2.7): now also Y1.1
- net at U3.27 (TA0.1/XIN/P2.6): now also Y1.2
- net at R29.1, U5.5 (+): now also J10.1 (Pin_1), TP11.1
- net at U4.7: now also C19.1, R43.2, TP7.1; no longer U4.6 (-)
- net at R29.2, U5.7: now also C21.1, TP15.1; no longer C20.1
- net at R26.2: now also J12.3 (Pin_3)
- net MSP_BSL_TX renamed MODULE_3_IN
- new net: D9.2 (A), R46.2
- new net: D8.2 (A), R44.1
- new net: J6.1 (Pin_1), R43.1, TP6.1, U4.5 (+)
- new net: D11.2 (A), R34.2
- new net: Q6.3 (D), R42.1
- new net: J6.3 (Pin_3), R42.2
- new net: D10.2 (A), R48.1
- new net: Q6.1 (G), R7.2, R8.2
- no-connect marks 23 -> 16
Other:
- moved on the sheet: C10, C12, C15, C16, C17, C7, Q1, Q3, Q4, Q5, R11, R17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

Commit message: board layout
Parts:
- removed D2: LED, LED_SMD:LED_0603_1608Metric_Pad1.05x0.95mm_HandSolder, symbol Device:LED
- removed J7: Screw_Terminal_01x08, symbol Connector:Screw_Terminal_01x08
- removed R34: 470R, symbol Device:R_Small
- removed R6: 470R, Resistor_SMD_AKL:R_0603_1608Metric_Pad1.05x0.95mm_HandSolder, symbol Device:R_Small
- removed TP1, TP11, TP12, TP13, TP15, TP16, TP17, TP19, TP2, TP20, TP21, TP3, TP6, TP7, TP8: TestPoint, TestPoint:TestPoint_Pad_D1.5mm, symbol Connector:TestPoint
- removed TP10: TestPoint, symbol Connector:TestPoint
- removed unit 4 of U5
- removed unit 3 of U5
- added D10: LED, LED_SMD:LED_0603_1608Metric_Pad1.05x0.95mm_HandSolder, symbol Device:LED
- added H1, H2, H3: MountingHole, MountingHole:MountingHole_3.2mm_M3_DIN965, symbol Mechanical:MountingHole
- added J5: Screw_Terminal_01x07, TerminalBlock_RND:TerminalBlock_RND_205-00006_1x07_P5.00mm_Horizontal, symbol Connector:Screw_Terminal_01x07
- added R25, R28: 470R, Resistor_SMD_AKL:R_0603_1608Metric_Pad1.05x0.95mm_HandSolder, symbol Device:R_Small
- added TP2: TestPoint, TestPoint:TestPoint_Pad_D1.5mm, symbol 4ms_Connector:TestPoint
- added unit 4 of U2
- added unit 3 of U2
- C18: renamed from C12; symbol Device:C_Small -> Device:C_Polarized_Small
- C5: renamed from C1; footprint Capacitor_THT_AKL:CP_Radial_D12.5mm_P5.00mm -> Capacitor_THT_AKL:CP_Radial_D10.0mm_P5.00mm
- D11: footprint (none) -> LED_SMD:LED_0603_1608Metric_Pad1.05x0.95mm_HandSolder
- J1: footprint Resistor_SMD_AKL:R_0603_1608Metric_Pad1.05x0.95mm_HandSolder -> TerminalBlock_RND:TerminalBlock_RND_205-00001_1x02_P5.00mm_Horizontal
- TP1: renamed from TP4; footprint (none) -> TestPoint:TestPoint_Pad_D1.5mm
- TP10: renamed from TP9; footprint (none) -> TestPoint:TestPoint_Pad_D1.5mm
- TP3: renamed from TP5; footprint (none) -> TestPoint:TestPoint_Pad_D1.5mm
- TP6: renamed from TP22; footprint (none) -> TestPoint:TestPoint_Pad_D1.5mm
- TP7: renamed from TP23; footprint (none) -> TestPoint:TestPoint_Pad_D1.5mm
- TP8: renamed from TP24; footprint (none) -> TestPoint:TestPoint_Pad_D1.5mm
- TP9: renamed from TP25; footprint (none) -> TestPoint:TestPoint_Pad_D1.5mm
- U1: footprint Package_SO_AKL:SOIC-8-1EP_3.9x4.9mm_P1.27mm_EP2.514x3.2mm -> Package_TO_SOT_SMD:TSOT-23-6_HandSoldering
- renumbered C3 to C1, C8 to C10, C21 to C11, C16 to C12, C17 to C13, C9 to C14, C11 to C15, C7 to C16, C10 to C17, C22 to C19, C4 to C2, C15 to C20, C23 to C21, C18 to C22, C19 to C23, C5 to C3, C6 to C4, C2 to C6, C20 to C7, C13 to C8, C14 to C9, D3 to D1, D1 to D2, D9 to D3, D10 to D9, J8 to J10, J6 to J11, J9 to J2, J4 to J3, J10 to J4, J11 to J6, J2 to J7, J3 to J8, J12 to J9, Q2 to Q1, Q3 to Q2, Q4 to Q3, Q5 to Q4, Q1 to Q5, R18 to R1, R14 to R10, R35 to R11, R15 to R12, R3 to R13, R4 to R14, R9 to R15, R39 to R16, R16 to R17, R10 to R18, R20 to R19, R12 to R2, R29 to R20, R44 to R21, R24 to R22, R36 to R23, R48 to R24, R40 to R26, R21 to R27, R30 to R29, R1 to R3, R25 to R30, R5 to R31, R45 to R32, R11 to R33, R47 to R34, R41 to R35, R37 to R36, R31 to R37, R26 to R38, R49 to R39, R46 to R4, R38 to R40, R8 to R41, R17 to R42, R7 to R43, R27 to R44, R22 to R45, R43 to R46, R42 to R47, R32 to R48, R33 to R49, R19 to R5, R2 to R6, R13 to R7, R28 to R8, R23 to R9, TP14 to TP4, TP18 to TP5, U5 to U2, U2 to U3, U3 to U5
Connections:
- net MODULE_3_IN is gone; now on net MODULE1_IN: J8.3 (Pin_3)
- net +3V3: now also R25.2, R28.2
- net GND: now also J5.7 (Pin_7), U2.13 (-), U2.9 (-)
- net GP_BUTTON: now also U5.15 (P3.4/TA0.0); no longer U5.21 (P3.7/TA1CLK/CAOUT)
- net GP_LED: now also U5.19 (P3.5/TA0.1); no longer D11.1 (K), U5.20 (P3.6/TA0.2)
- net MODULE1_IN: now also U5.7 (TMS/TA0.0/UCB0CLK/UCA0STE/A5/CA5/P1.5); no longer U5.5 (ADC10CLK/CAOUT/VREF-/VeREF-/A3/CA3/P1.3)
- net MODULE1_OUT: now also U5.16 (TA1.0/P2.3), TP2.1; no longer U5.10 (TA1.0/P2.0)
- net MODULE1_STATUS: now also U5.11 (TA1.1/P2.1), J5.1 (Pin_1); no longer U5.9 (P3.0/TA0.2)
- net MODULE2_IN: now also U5.5 (ADC10CLK/CAOUT/VREF-/VeREF-/A3/CA3/P1.3); no longer U5.6 (TCK/SMCLK/UCB0STE/UCA0CLK/VREF+/VeREF+/A4/CA4/P1.4)
- net MODULE2_OUT: now also U5.14 (P3.3/TA1.2); no longer U5.11 (TA1.1/P2.1)
- net MODULE2_STATUS: now also U5.10 (TA1.0/P2.0), J5.2 (Pin_2); no longer U5.8 (P3.1/TA1.0)
- net MODULE3_IN: now also U5.6 (TCK/SMCLK/UCB0STE/UCA0CLK/VREF+/VeREF+/A4/CA4/P1.4); no longer U5.7 (TMS/TA0.0/UCB0CLK/UCA0STE/A5/CA5/P1.5)
- net MODULE3_OUT: now also U5.18 (TA1.2/P2.5); no longer U5.12 (TA1.1/P2.2)
- net MODULE3_STATUS: now also U5.9 (P3.0/TA0.2), J5.3 (Pin_3); no longer U5.13 (P3.2/TA1.1)
- net MODULE4_IN: now also U5.2 (TA0CLK/ACLK/A0/CA0/P1.0); no longer U5.22 (TDI/TCLK/TA0.1/UCB0SOMI/UCB0SCL/A6/CA6/P1.6)
- net MODULE4_OUT: now also U5.13 (P3.2/TA1.1); no longer U5.16 (TA1.0/P2.3)
- net MODULE4_STATUS: now also U5.8 (P3.1/TA1.0), J5.4 (Pin_4); no longer U5.14 (P3.3/TA1.2)
- net MODULE5_IN: now also C23.2, R49.2; no longer C22.2, R48.2
- net MODULE5_OUT: now also R43.1; no longer R42.1
- net MODULE5_STATUS: now also U5.20 (P3.6/TA0.2), J5.5 (Pin_5); no longer U5.15 (P3.4/TA0.0)
- net MODULE6_IN: now also C22.2, R48.2, U5.22 (TDI/TCLK/TA0.1/UCB0SOMI/UCB0SCL/A6/CA6/P1.6); no longer C23.2, R49.2, U5.2 (TA0CLK/ACLK/A0/CA0/P1.0)
- net MODULE6_OUT: now also R42.1, U5.12 (TA1.1/P2.2); no longer R43.1, U5.18 (TA1.2/P2.5)
- net MODULE6_STATUS: now also U5.21 (P3.7/TA1CLK/CAOUT), J5.6 (Pin_6); no longer U5.19 (P3.5/TA0.1)
- net VUSB_SENSE: now also U3.19 (CBUS3); no longer U3.10 (CBUS2)
- net at C19.1, R29.2: now also U2.14
- net at J9.1 (Pin_1), R37.1: now also U2.10 (+)
- net at C21.1, R37.2: now also U2.8
- net at J6.1 (Pin_1), R29.1: now also U2.12 (+)
- net at D11.2 (A): now also R28.1
- net FT_USB+: now reaches R14.2, U3.11 (USBDP)
- net FT_USB-: now reaches R13.2, U3.12 (USBDM)
- net TX_LED: now reaches U3.17 (CBUS1)
- net TX_LED: now also D11.1 (K)
- net RX_LED: now reaches U3.18 (CBUS0)
- net RX_LED: now also D10.1 (K)
- new net: D10.2 (A), R25.1
- no-connect marks 16 -> 15
Other:
- moved on the sheet: C10

Commit message: finished hardware revision 1.0
Parts:
- renumbered C5 to C1, C20 to C10, C1 to C11, C2 to C12, C22 to C13, C10 to C14, C3 to C15, C4 to C16, C12 to C17, C23 to C18, C13 to C19, C8 to C2, C7 to C20, C11 to C21, C19 to C22, C21 to C23, C14 to C3, C6 to C4, C16 to C5, C15 to C6, C9 to C7, C17 to C8, C18 to C9, D2 to D1, D8 to D10, D9 to D11, D10 to D2, D11 to D3, D3 to D4, D1 to D5, D4 to D6, D5 to D7, D6 to D8, D7 to D9, J6 to J10, J9 to J11, J7 to J2, J8 to J3, J10 to J4, J3 to J5, J11 to J6, J5 to J7, J2 to J8, J4 to J9, Q5 to Q1, Q6 to Q2, Q1 to Q3, Q2 to Q4, Q3 to Q5, Q4 to Q6, R42 to R1, R48 to R10, R25 to R11, R28 to R12, R4 to R13, R15 to R14, R18 to R15, R33 to R16, R43 to R17, R41 to R18, R47 to R19, R40 to R2, R46 to R20, R49 to R21, R34 to R22, R2 to R23, R7 to R24, R10 to R25, R12 to R26, R17 to R27, R21 to R28, R24 to R29, R13 to R3, R5 to R30, R19 to R31, R27 to R32, R36 to R33, R1 to R34, R16 to R35, R26 to R36, R35 to R37, R9 to R38, R22 to R39, R14 to R4, R30 to R40, R38 to R41, R8 to R42, R20 to R43, R29 to R44, R37 to R45, R11 to R46, R23 to R47, R32 to R48, R39 to R49, R45 to R5, R31 to R6, R44 to R7, R3 to R8, R6 to R9, TP5 to TP10, TP3 to TP2, TP6 to TP3, TP7 to TP4, TP8 to TP5, TP9 to TP6, TP10 to TP7, TP2 to TP8, TP4 to TP9, U4 to U2, U5 to U4, U2 to U5
Connections:
- net at Y1.1: now also U4.27 (TA0.1/XIN/P2.6); no longer U4.26 (XOUT/P2.7)
- net at Y1.2: now also U4.26 (XOUT/P2.7); no longer U4.27 (TA0.1/XIN/P2.6)
Other:
- moved on the sheet: C14, C17, C19, C2, C3, C5, C6, C7, C8, C9, D2, D3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

Commit message: finished hardware rev 1.1
Parts:
- removed J3: BSL_SEL, Connector_PinHeader_2.54mm:PinHeader_1x03_P2.54mm_Vertical, symbol Connector_Generic:Conn_01x03
- removed J7: Screw_Terminal_01x07, TerminalBlock_RND:TerminalBlock_RND_205-00006_1x07_P5.00mm_Horizontal, symbol Connector:Screw_Terminal_01x07
- removed R16: 330R, Resistor_SMD_AKL:R_0603_1608Metric_Pad1.05x0.95mm_HandSolder, symbol Device:R_Small
- removed R45: 470k, Resistor_SMD_AKL:R_0603_1608Metric_Pad1.05x0.95mm_HandSolder, symbol Device:R_Small
- added J3: BSL_SEL, Connector_PinHeader_2.54mm:PinHeader_2x03_P2.54mm_Vertical, symbol Connector_Generic:Conn_02x03_Odd_Even
- added J7: Screw_Terminal_01x08, TerminalBlock_RND:TerminalBlock_RND_205-00007_1x08_P5.00mm_Horizontal, symbol Connector:Screw_Terminal_01x08
- added JP1: Jumper_2_Open, 4ms_SolderJumper:JUMPER_SMD_1x2, symbol Jumper:Jumper_2_Open
- added R16, R45: 10k, Resistor_SMD_AKL:R_0603_1608Metric_Pad1.05x0.95mm_HandSolder, symbol Device:R
- added R50: 470k, Resistor_SMD_AKL:R_0603_1608Metric_Pad1.05x0.95mm_HandSolder, symbol Device:R_Small
- added SW2: SW_Push, Button_Switch_THT:SW_PUSH_6mm, symbol Switch:SW_Push
- added TP11: TestPoint, TestPoint:TestPoint_Pad_1.5x1.5mm, symbol 4ms_Connector:TestPoint
- added TP12, TP13: TestPoint, TestPoint:TestPoint_Pad_D1.5mm, symbol 4ms_Connector:TestPoint
- C10: value 2n2 -> 1n
- U2: footprint Package_SO_AKL:SOIC-8-1EP_3.9x4.9mm_P1.27mm_EP2.514x3.2mm -> Package_SO_AKL:SOIC-8_3.9x4.9mm_P1.27mm
Connections:
- net 3V3OUT is gone; now on net +3V3: C14.1, U3.13 (3V3OUT), U3.14 (~{RESET}), U3.3 (VCCIO)
- net +3V3: now also J7.1 (Pin_1), TP12.1
- net FT231_DTR#: now also R45.1; no longer C10.1, J2.1 (Pin_1), R6.2, U4.24 (~{RST}/NMI/SBWTDIO)
- net FT231_RTS#: now also R16.1; no longer J2.8 (Pin_8), U4.25 (SBWTCK/TEST)
- net FT231_RX: now also J3.3 (Pin_3)
- net FT231_TX: now also J3.4 (Pin_4); no longer U4.3 (TA0.0/UCA0RXD/UCA0SOMI/A1/CA1/P1.1)
- net GND: now also U2.3 (+), U2.5 (+), U5.10 (+), U5.12 (+), U5.3 (+), U5.5 (+), J7.8 (Pin_8), JP1.1 (A), SW2.1, TP11.1, TP13.1; no longer D10.1 (K), D5.1 (K), D6.1 (K), D7.1 (K), D8.1 (K), D9.1 (K), U2.2 (-), U2.6 (-), U5.13 (-), U5.2 (-), U5.6 (-), U5.9 (-)
- net MODULE1_IN: now also J3.6 (Pin_6)
- net MODULE1_OUT: now also U4.11 (TA1.1/P2.1); no longer U4.16 (TA1.0/P2.3)
- net MODULE1_STATUS: now also U4.10 (TA1.0/P2.0), J7.2 (Pin_2); no longer U4.11 (TA1.1/P2.1)
- net MODULE2_STATUS: now also U4.9 (P3.0/TA0.2), J7.3 (Pin_3); no longer U4.10 (TA1.0/P2.0)
- net MODULE3_OUT: now also U4.17 (TA1.2/P2.4); no longer U4.18 (TA1.2/P2.5)
- net MODULE3_STATUS: now also U4.8 (P3.1/TA1.0), J7.4 (Pin_4); no longer U4.9 (P3.0/TA0.2)
- net MODULE4_STATUS: now also U4.16 (TA1.0/P2.3), J7.5 (Pin_5); no longer U4.8 (P3.1/TA1.0)
- net MODULE5_OUT: now also U4.18 (TA1.2/P2.5); no longer U4.17 (TA1.2/P2.4)
- net MODULE5_STATUS: now also J7.6 (Pin_6)
- net MODULE6_STATUS: now also J7.7 (Pin_7)
- net MSP_UART_TX: now also J3.1 (Pin_1)
- net TCK: now also U4.25 (SBWTCK/TEST), R16.2
- net at J8.1 (Pin_1), R42.1: now also U5.2 (-); no longer U5.3 (+)
- net at J11.1 (Pin_1): now also R44.1, U5.9 (-); no longer U5.10 (+)
- net at C23.1, U5.8: now also R44.2
- net at C22.1, U5.14: now also R43.2; no longer R44.2
- net at J4.1 (Pin_1), R7.1: now also U2.2 (-); no longer U2.3 (+)
- net at C21.1, U5.7: now also R50.2; no longer R43.2
- net at J6.1 (Pin_1), R20.1: now also U2.6 (-); no longer U2.5 (+)
- new net: J10.1 (Pin_1), R43.1, U5.13 (-)
- new net: D10.1 (K), D5.1 (K), D6.1 (K), D7.1 (K), D8.1 (K), D9.1 (K), JP1.2 (B)
- new net: J9.1 (Pin_1), R50.1, U5.6 (-)
- new net MSP_UART_RX: J3.2 (Pin_2), J3.5 (Pin_5), U4.3 (TA0.0/UCA0RXD/UCA0SOMI/A1/CA1/P1.1)
- new net TDO/TDI: C10.1, J2.1 (Pin_1), R45.2, R6.2, SW2.2, U4.24 (~{RST}/NMI/SBWTDIO)
- no-connect marks 15 -> 16
Other:
- title: (none) -> Infrared model train detector
- moved on the sheet: C14, R42, TP9
